File: rck.kicad_sch (KiCad schematic)
At the start: 53 parts, among them J1 Conn_02x22_Row_Letter_Last, J2 Conn_02x22_Row_Letter_Last, J3 Conn_02x22_Row_Letter_Last, J4 Conn_02x22_Row_Letter_Last, J5 Conn_02x22_Row_Letter_Last, J6 Conn_02x22_Row_Letter_Last, J7 Conn_01x06_Pin

Commit message: update 10F
Parts:
- added R19, R20, R21, R22, R23, R24, R25, R26, R27, R28, R29, R30: R, Resistor_SMD:R_1206_3216Metric, symbol Device:R
- added rD19, rD20, rD21, rD22, rD23, rD24, rD25, rD26, rD27, rD28, rD29, rD30: LED, LED_SMD:LED_1206_3216Metric, symbol Device:LED
Connections:
- net +5V: no longer J1.1a (Pin_1a)
- net VCC: now also J1.1a (Pin_1a), R19.2, R20.2, R21.2, R22.2, R23.2, R24.2, R25.2, R26.2, R27.2, R28.2, R29.2, R30.2
- net F5-01: now reaches J1.14a (Pin_14a), J4.2a (Pin_2a), rD13.1 (K)
- net F3-03: now reaches J1.10a (Pin_10a), J3.10a (Pin_10a), rD9.1 (K)
- net F1-02: now reaches J1.3a (Pin_3a), J2.6a (Pin_6a), rD2.1 (K)
- net F4-02: now reaches J1.12a (Pin_12a), J3.18a (Pin_18a), rD11.1 (K)
- net F3-01: now reaches J1.8a (Pin_8a), J3.2a (Pin_2a), rD7.1 (K)
- net F5-03: now reaches J1.16a (Pin_16a), J4.10a (Pin_10a), rD15.1 (K)
- net F6-01: now reaches J1.17a (Pin_17a), J4.14a (Pin_14a), rD16.1 (K)
- net F6-02: now reaches J1.18a (Pin_18a), J4.18a (Pin_18a), rD17.1 (K)
- net F6-03: now reaches J1.19a (Pin_19a), J4.22a (Pin_22a), rD18.1 (K)
- net F5-02: now reaches J1.15a (Pin_15a), J4.6a (Pin_6a), rD14.1 (K)
- net F4-01: now reaches J1.11a (Pin_11a), J3.14a (Pin_14a), rD10.1 (K)
- net F4-03: now reaches J1.13a (Pin_13a), J3.22a (Pin_22a), rD12.1 (K)
- net F3-02: now reaches J1.9a (Pin_9a), J3.6a (Pin_6a), rD8.1 (K)
- net F1-03: now reaches J1.4a (Pin_4a), J2.10a (Pin_10a), rD3.1 (K)
- net F1-01: now reaches J1.2a (Pin_2a), J2.2a (Pin_2a), rD1.1 (K)
- net F2-03: now reaches J1.7a (Pin_7a), J2.22a (Pin_22a), rD6.1 (K)
- net F2-01: now reaches J1.5a (Pin_5a), J2.14a (Pin_14a), rD4.1 (K)
- net F2-02: now reaches J1.6a (Pin_6a), J2.18a (Pin_18a), rD5.1 (K)
- net F7-01: now reaches J1.20a (Pin_20a)
- net F7-01: now also J5.2a (Pin_2a), rD19.1 (K)
- net F7-02: now reaches J1.21a (Pin_21a)
- net F7-02: now also J5.6a (Pin_6a), rD20.1 (K)
- net A5-01 renamed F7-03
- net F7-03: now also J5.10a (Pin_10a), rD21.1 (K); no longer J5.2a (Pin_2a)
- net A5-02 renamed F8-01
- net F8-01: now also J5.14a (Pin_14a), rD22.1 (K); no longer J5.6a (Pin_6a)
- net A5-03 renamed F8-02
- net F8-02: now also J5.18a (Pin_18a), rD23.1 (K); no longer J5.10a (Pin_10a)
- net A5-04 renamed F8-03
- net F8-03: now also J5.22a (Pin_22a), rD24.1 (K); no longer J5.14a (Pin_14a)
- net A5-05 renamed F9-01
- net F9-01: now also J6.2a (Pin_2a), rD25.1 (K); no longer J5.18a (Pin_18a)
- net A5-06 renamed F9-02
- net F9-02: now also J6.6a (Pin_6a), rD26.1 (K); no longer J5.22a (Pin_22a)
- net A6-01 renamed F9-03
- net F9-03: now also J6.10a (Pin_10a), rD27.1 (K); no longer J6.2a (Pin_2a)
- net A6-02 renamed F10-01
- net F10-01: now also J6.14a (Pin_14a), rD28.1 (K); no longer J6.6a (Pin_6a)
- net A6-03 renamed F10-02
- net F10-02: now also J6.18a (Pin_18a), rD29.1 (K); no longer J6.10a (Pin_10a)
- net A6-04 renamed F10-03
- net F10-03: now also J6.22a (Pin_22a), rD30.1 (K); no longer J6.14a (Pin_14a)
- net A6-05: no longer names the net of J1.11b (Pin_11b)
- net A6-05: no longer J6.18a (Pin_18a)
- net A6-06: no longer names the net of J1.12b (Pin_12b)
- net A6-06: no longer J6.22a (Pin_22a)
- new net: R24.1, rD24.2 (A)
- new net: R20.1, rD20.2 (A)
- new net: R29.1, rD29.2 (A)
- new net: R30.1, rD30.2 (A)
- new net: R26.1, rD26.2 (A)
- new net: R28.1, rD28.2 (A)
- new net: R27.1, rD27.2 (A)
- new net: R25.1, rD25.2 (A)
- new net: R21.1, rD21.2 (A)
- new net: R22.1, rD22.2 (A)
- new net: R23.1, rD23.2 (A)
- new net: R19.1, rD19.2 (A)
Other:
- moved on the sheet: C1, C2, C3, C4, C5, C6, C7, C8, J1, J2, J3, J4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

Commit message: 10F
Connections:
- net +5V: now also J1.1a (Pin_1a)
- net VCC: no longer J1.1a (Pin_1a)
Changed lines of the file:
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@@
 		)
 	)
-	(label "VCC"
+	(label "+5V"
 		(at 215.9 88.9 0)
 		(fields_autoplaced yes)
