File: rck.kicad_sch (KiCad schematic)
At the start: 68 parts, among them J1 Conn_02x22_Row_Letter_Last, J2 Conn_02x22_Row_Letter_Last, J3 Conn_02x22_Row_Letter_Last, J4 Conn_02x22_Row_Letter_Last, J5 Conn_02x22_Row_Letter_Last, J7 Conn_01x02_Pin

Commit message: 6F Complete
Parts:
- removed J5: Conn_02x22_Row_Letter_Last, Library:Edac_22x2_3.96, symbol Connector_Generic:Conn_02x22_Row_Letter_Last
- removed R19, R20, R21, R22, R23, R24: R, Resistor_SMD:R_1206_3216Metric, symbol Device:R
- removed rD19, rD20, rD21, rD22, rD23, rD24: LED, LED_SMD:LED_1206_3216Metric, symbol Device:LED
Connections:
- net F7-01: no longer names the net of J1.20a (Pin_20a)
- net F7-02: no longer names the net of J1.21a (Pin_21a)
- net F7-03: no longer names the net of J1.1b (Pin_1b)
- net F8-01: no longer names the net of J1.2b (Pin_2b)
- net F8-02: no longer names the net of J1.3b (Pin_3b)
- net F8-03: no longer names the net of J1.4b (Pin_4b)
Other:
- moved on the sheet: R1, R10, R11, R12, R13, R14, R15, R16, R17, R18, R2, R3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
