File: rck.kicad_sch (KiCad schematic)
At the start: 77 parts, among them J1 Conn_02x22_Row_Letter_Last, J2 Conn_02x22_Row_Letter_Last, J3 Conn_02x22_Row_Letter_Last, J4 Conn_02x22_Row_Letter_Last, J5 Conn_02x22_Row_Letter_Last, J6 Conn_02x22_Row_Letter_Last, J7 Conn_01x06_Pin

Commit message: F10 Compleate
Parts:
- removed J7: Conn_01x06_Pin, Connector_PinSocket_2.54mm:PinSocket_1x06_P2.54mm_Vertical, symbol Connector:Conn_01x06_Pin
- added Brd1: SSD1306, SSD1306:128x64OLED, symbol SSD1306-128x64_OLED:SSD1306
- added F1: SMD0805-020-16V - 2.8A, Fuse:Fuse_0805_2012Metric, symbol Device:Fuse_Small
- added F2: SMD0805-020-16V - 500mA, Fuse:Fuse_0805_2012Metric, symbol Device:Fuse_Small
- added F3: SMD0603-050 - 1A, Fuse:Fuse_0603_1608Metric, symbol Device:Fuse_Small
- added J7: Conn_01x02_Pin, Connector_PinSocket_2.54mm:PinSocket_1x02_P2.54mm_Vertical, symbol Connector:Conn_01x02_Pin
Connections:
- net +12V: now also F1.2, J7.1 (Pin_1); no longer C1.1, C2.2, C5.1, C6.2, VR1.1 (Vin), VR2.1 (Vin)
- net +5V: now also F3.2; no longer C7.1, C8.2, VR2.3 (Vout)
- net GND: now also Brd1.1 (GND), J7.2 (Pin_2)
- net VCC: now also F2.2; no longer C3.1, C4.2, VR1.3 (Vout)
- net 3V: now reaches J1.20b (Pin_20b)
- net 3V: now also Brd1.2 (VCC)
- net SDA: now reaches J1.21b (Pin_21b)
- net SDA: now also Brd1.4 (SDA)
- net SCL: now reaches J1.22b (Pin_22b)
- net SCL: now also Brd1.3 (SCL)
- new net: C1.1, C2.2, C5.1, C6.2, F1.1, VR1.1 (Vin), VR2.1 (Vin)
- new net: C7.1, C8.2, F3.1, VR2.3 (Vout)
- new net: C3.1, C4.2, F2.1, VR1.3 (Vout)
Other:
- moved on the sheet: C1, C2, C3, C4, C5, C6, C7, C8, VR1, VR2

Commit message: update
Other:
- note added: "Modulo de Potencia"
- moved on the sheet: Brd1, C1, C2, C3, C4, C5, C6, C7, C8, F1, F2, F3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
