File: rck.kicad_pcb (KiCad board)
At the start: 2 copper layers, 150 x 285.6 mm, 69 parts, among them J1 Conn_02x22_Row_Letter_Last, J2 Conn_02x22_Row_Letter_Last, J3 Conn_02x22_Row_Letter_Last, J4 Conn_02x22_Row_Letter_Last, J5 Conn_02x22_Row_Letter_Last, J7 Conn_01x02_Pin

Commit message: Fix route
Routing:
- net /F6-01: track 194.5 -> 193.8 mm
- net GND: vias 38 -> 39
Changed lines of the file:
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@@
 	)
 	(via
+		(at 214.14746 123.323)
+		(size 0.8)
+		(drill 0.4)
+		(layers "F.Cu" "B.Cu")
+		(free yes)
+		(net 2)
+	)
+	(via
 		(at 124.79746 218.373)
 		(size 0.8)
@@
 	)
 	(via
-		(at 181.24746 123.723)
+		(at 181.29746 123.273)
 		(size 0.8)
 		(drill 0.4)
@@
 	)
 	(segment
-		(start 216.95246 120.713)
-		(end 216.95246 122.018)
+		(start 214.99746 118.758)
+		(end 216.95246 120.713)
 		(width 0.25)
 		(layer "B.Cu")
@@
 	)
 	(segment
-		(start 131.59746 252.373)
-		(end 147.79746 268.573)
+		(start 174.23104 268.573)
+		(end 181.29104 275.633)
 		(width 0.25)
 		(layer "B.Cu")
@@
 	)
 	(segment
-		(start 214.99746 118.758)
-		(end 216.95246 120.713)
+		(start 216.95246 120.713)
+		(end 216.95246 122.018)
 		(width 0.25)
 		(layer "B.Cu")
@@
 	)
 	(segment
-		(start 174.23104 268.573)
-		(end 181.29104 275.633)
+		(start 153.772155 131.173)
+		(end 131.59746 153.347695)
 		(width 0.25)
 		(layer "B.Cu")
@@
 	)
 	(segment
-		(start 207.99746 130.973)
-		(end 153.972155 130.973)
+		(start 131.59746 252.373)
+		(end 147.79746 268.573)
 		(width 0.25)
 		(layer "B.Cu")
@@
 	)
 	(segment
-		(start 216.95246 122.018)
-		(end 207.99746 130.973)
+		(start 207.79746 131.173)
+		(end 153.772155 131.173)
 		(width 0.25)
 		(layer "B.Cu")
@@
 	)
 	(segment
-		(start 147.79746 268.573)
-		(end 174.23104 268.573)
+		(start 199.79746 91.073)
+		(end 209.99746 91.073)
 		(width 0.25)
 		(layer "B.Cu")
@@
 	)
 	(segment
-		(start 199.79746 91.073)
-		(end 209.99746 91.073)
+		(start 214.99746 96.073)
+		(end 214.99746 118.758)
 		(width 0.25)
 		(layer "B.Cu")
@@
 	)
 	(segment
-		(start 131.59746 153.347695)
-		(end 131.59746 252.373)
+		(start 209.99746 91.073)
+		(end 214.99746 96.073)
 		(width 0.25)
 		(layer "B.Cu")
@@
 	)
 	(segment
-		(start 214.99746 96.073)
-		(end 214.99746 118.758)
+		(start 216.95246 122.018)
+		(end 207.79746 131.173)
 		(width 0.25)
 		(layer "B.Cu")
@@
 	)
 	(segment
-		(start 209.99746 91.073)
-		(end 214.99746 96.073)
+		(start 131.59746 153.347695)
+		(end 131.59746 252.373)
 		(width 0.25)
 		(layer "B.Cu")
@@
 	)
 	(segment
-		(start 153.972155 130.973)
-		(end 131.59746 153.347695)
+		(start 147.79746 268.573)
+		(end 174.23104 268.573)
 		(width 0.25)
 		(layer "B.Cu")
@@
 	)
 	(segment
-		(start 156.99746 180.973)
-		(end 155.49746 182.473)
-		(width 0.25)
-		(layer "B.Cu")
-		(net 45)
-	)
-	(segment
 		(start 156.99746 165.473)
-		(end 156.99746 180.973)
+		(end 155.54746 164.023)
 		(width 0.25)
 		(layer "B.Cu")
@@
 	)
 	(segment
-		(start 156.39746 147.173)
-		(end 155.54746 148.023)
+		(start 155.81438 113.373)
+		(end 153.55438 115.633)
 		(width 0.25)
 		(layer "B.Cu")
@@
 	)
 	(segment
-		(start 155.54746 148.023)
-		(end 155.54746 164.023)
+		(start 165.29746 106.373)
+		(end 158.29746 113.373)
 		(width 0.25)
 		(layer "B.Cu")
@@
 	)
 	(segment
-		(start 155.81438 113.373)
-		(end 153.55438 115.633)
+		(start 156.99746 180.973)
+		(end 156.99746 165.473)
 		(width 0.25)
 		(layer "B.Cu")
@@
 	)
 	(segment
-		(start 165.29746 106.373)
-		(end 158.29746 113.373)
+		(start 155.54746 146.323)
+		(end 155.49746 146.273)
 		(width 0.25)
 		(layer "B.Cu")
@@
 	)
 	(segment
-		(start 155.54746 164.023)
-		(end 156.99746 165.473)
+		(start 158.29746 113.373)
+		(end 155.81438 113.373)
 		(width 0.25)
 		(layer "B.Cu")
@@
 	)
 	(segment
-		(start 155.49746 146.273)
-		(end 156.39746 147.173)
+		(start 155.49746 182.473)
+		(end 156.99746 180.973)
 		(width 0.25)
 		(layer "B.Cu")
@@
 	)
 	(segment
-		(start 158.29746 113.373)
-		(end 155.81438 113.373)
+		(start 155.54746 164.023)
+		(end 155.54746 146.323)
 		(width 0.25)
 		(layer "B.Cu")
@@
 	)
 	(segment
-		(start 146.39746 125.573)
+		(start 146.59746 125.373)
 		(end 119.99746 151.973)
 		(width 0.25)
@@
 	)
 	(segment
-		(start 187.29746 125.573)
-		(end 146.39746 125.573)
-		(width 0.25)
-		(layer "B.Cu")
-		(net 208)
-	)
-	(segment
-		(start 189.2158 123.65466)
-		(end 187.29746 125.573)
+		(start 189.2158 120.713)
+		(end 189.2158 123.65466)
 		(width 0.25)
 		(layer "B.Cu")
@@
 	)
 	(segment
-		(start 189.2158 120.713)
-		(end 189.2158 123.65466)
+		(start 187.49746 125.373)
+		(end 146.59746 125.373)
+		(width 0.25)
+		(layer "B.Cu")
+		(net 208)
+	)
+	(segment
+		(start 189.2158 123.65466)
+		(end 187.49746 125.373)
 		(width 0.25)
 		(layer "B.Cu")
@@
 	)
 	(segment
-		(start 183.79746 124.773)
-		(end 145.79746 124.773)
+		(start 185.25342 120.713)
+		(end 185.25342 123.31704)
 		(width 0.25)
 		(layer "B.Cu")
@@
 	(segment
 		(start 185.25342 123.31704)
-		(end 183.79746 124.773)
+		(end 183.99746 124.573)
 		(width 0.25)
 		(layer "B.Cu")
@@
 	)
 	(segment
-		(start 185.25342 120.713)
-		(end 185.25342 123.31704)
+		(start 183.99746 124.573)
+		(end 145.99746 124.573)
 		(width 0.25)
 		(layer "B.Cu")
@@
 	)
 	(segment
-		(start 145.79746 124.773)
+		(start 145.99746 124.573)
 		(end 119.29746 151.273)
 		(width 0.25)
@@
 		(name "$teardrop_padvia$")
 		(hatch full 0.1)
-		(priority 30001)
+		(priority 30002)
 		(attr
 			(teardrop
@@
 		(polygon
 			(pts
-				(xy 136.473504 96.795703) (xy 136.296727 96.618926) (xy 135.666357 96.903448) (xy 135.818723 97.273707)
-				(xy 136.188982 97.426073)
-			)
-		)
-	)
-	(zone
-		(net 2)
-		(net_name "GND")
-		(layer "F.Cu")
-		(hatch edge 0.5)
-		(priority 1)
-		(connect_pads
-			(clearance 0.5)
-		)
-		(min_thickness 0.25)
-		(filled_areas_thickness no)
-		(fill yes
-			(thermal_gap 0.5)
-			(thermal_bridge_width 0.5)
-		)
-		(polygon
-			(pts
-				(xy 100.39746 35.073) (xy 250.29746 35.123) (xy 250.39746 320.573) (xy 100.39746 320.573)
+				(xy 135.63037 83.293) (xy 135.63037 83.543) (xy 136.266357 83.842552) (xy 136.42043 83.473) (xy 136.266357 83.103448)
 			)
 		)
@@
 		(name "$teardrop_padvia$")
 		(hatch full 0.1)
-		(priority 30002)
+		(priority 30001)
 		(attr
 			(teardrop
@@
 		(polygon
 			(pts
-				(xy 135.63037 83.293) (xy 135.63037 83.543) (xy 136.266357 83.842552) (xy 136.42043 83.473) (xy 136.266357 83.103448)
+				(xy 136.473504 96.795703) (xy 136.296727 96.618926) (xy 135.666357 96.903448) (xy 135.818723 97.273707)
+				(xy 136.188982 97.426073)
 			)
 		)
@@
 			)
 		)
+	)
+	(zone
+		(net 2)
+		(net_name "GND")
+		(layer "F.Cu")
+		(hatch edge 0.5)
+		(priority 1)
+		(connect_pads
+			(clearance 0.5)
+		)
+		(min_thickness 0.25)
+		(filled_areas_thickness no)
+		(fill yes
+			(thermal_gap 0.5)
+			(thermal_bridge_width 0.5)
+		)
+		(polygon
+			(pts
+				(xy 100.39746 35.073) (xy 250.29746 35.123) (xy 250.39746 320.573) (xy 100.39746 320.573)
+			)
+		)

Commit message: Fix routes
Parts:
- moved C1 2.77 mm to (114.3, 107.6)
- moved C2 0.93 mm to (123.2, 108.5)
Routing:
- net /3V: track 191.8 -> 187.1 mm
- net /SCL: track 176.4 -> 172.4 mm
- net /SDA: track 190.9 -> 187.3 mm
Changed lines of the file:
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@@
 	(footprint "Capacitor_SMD:C_1210_3225Metric"
 		(layer "B.Cu")
-		(at 123.49746 109.373 90)
+		(at 123.24746 108.473 90)
 		(descr "Capacitor SMD 1210 (3225 Metric), square (rectangular) end terminal, IPC_7351 nominal, (Body size source: IPC-SM-782 page 76, https://www.pcb-3d.com/wordpress/wp-content/uploads/ipc-sm-782a_amendment_1_and_2.pdf), generated with kicad-footprint-generator")
 		(tags "capacitor")
@@
 	(footprint "Capacitor_SMD:CP_Elec_5x5.9"
 		(layer "B.Cu")
-		(at 115.59746 110.073 -90)
+		(at 114.29746 107.623 -90)
 		(descr "SMD capacitor, aluminum electrolytic, Panasonic B6, 5.0x5.9mm")
 		(tags "capacitor electrolytic")
@@
 	)
 	(segment
-		(start 107.69746 117.073)
-		(end 107.69746 45.873)
+		(start 132.73746 120.713)
+		(end 131.27246 119.248)
 		(width 0.25)
 		(layer "B.Cu")
@@
 	)
 	(segment
-		(start 174.99746 37.573)
-		(end 176.50746 39.083)
+		(start 133.74246 120.713)
+		(end 132.73746 120.713)
 		(width 0.25)
 		(layer "B.Cu")
@@
 	)
 	(segment
-		(start 115.39746 124.773)
-		(end 107.69746 117.073)
+		(start 107.69746 110.798)
+		(end 107.69746 45.873)
 		(width 0.25)
 		(layer "B.Cu")
@@
 	)
 	(segment
-		(start 129.68246 124.773)
-		(end 115.39746 124.773)
+		(start 131.27246 119.248)
+		(end 131.27246 113.948)
 		(width 0.25)
 		(layer "B.Cu")
@@
 	)
 	(segment
-		(start 133.74246 120.713)
-		(end 129.68246 124.773)
+		(start 174.99746 37.573)
+		(end 176.50746 39.083)
+		(width 0.25)
+		(layer "B.Cu")
+		(net 24)
+	)
+	(segment
+		(start 129.69746 112.373)
+		(end 109.27246 112.373)
+		(width 0.25)
+		(layer "B.Cu")
+		(net 24)
+	)
+	(segment
+		(start 109.27246 112.373)
+		(end 107.69746 110.798)
+		(width 0.25)
+		(layer "B.Cu")
+		(net 24)
+	)
+	(segment
+		(start 131.27246 113.948)
+		(end 129.69746 112.373)
 		(width 0.25)
 		(layer "B.Cu")
@@
 	)
 	(segment
-		(start 112.79746 129.323)
-		(end 103.84746 120.373)
+		(start 130.92246 124.648)
+		(end 129.07246 122.798)
 		(width 0.25)
 		(layer "B.Cu")
@@
 	)
 	(segment
-		(start 103.84746 120.373)
+		(start 103.84746 111.673)
 		(end 103.84746 48.923)
 		(width 0.25)
@@
 	)
 	(segment
-		(start 133.05724 129.323)
-		(end 112.79746 129.323)
+		(start 129.07246 115.473)
+		(end 127.62246 114.023)
 		(width 0.25)
 		(layer "B.Cu")
@@
 	(segment
 		(start 141.66724 120.713)
-		(end 133.05724 129.323)
+		(end 137.73224 124.648)
+		(width 0.25)
+		(layer "B.Cu")
+		(net 36)
+	)
+	(segment
+		(start 127.62246 114.023)
+		(end 106.19746 114.023)
+		(width 0.25)
+		(layer "B.Cu")
+		(net 36)
+	)
+	(segment
+		(start 129.07246 122.798)
+		(end 129.07246 115.473)
+		(width 0.25)
+		(layer "B.Cu")
+		(net 36)
+	)
+	(segment
+		(start 137.73224 124.648)
+		(end 130.92246 124.648)
+		(width 0.25)
+		(layer "B.Cu")
+		(net 36)
+	)
+	(segment
+		(start 106.19746 114.023)
+		(end 103.84746 111.673)
 		(width 0.25)
 		(layer "B.Cu")
@@
 	)
 	(segment
-		(start 105.84746 118.973)
-		(end 105.84746 45.373)
+		(start 105.84746 45.373)
+		(end 114.49746 36.723)
 		(width 0.25)
 		(layer "B.Cu")
@@
 	)
 	(segment
-		(start 179.04746 38.623)
-		(end 179.04746 40.473)
+		(start 130.22246 121.698)
+		(end 130.22246 114.848)
 		(width 0.25)
 		(layer "B.Cu")
@@
 	)
 	(segment
-		(start 137.70486 120.713)
-		(end 131.24486 127.173)
+		(start 128.59746 113.223)
+		(end 107.69746 113.223)
 		(width 0.25)
 		(layer "B.Cu")
@@
 	)
 	(segment
-		(start 131.24486 127.173)
-		(end 114.04746 127.173)
+		(start 105.84746 111.373)
+		(end 105.84746 45.373)
 		(width 0.25)
 		(layer "B.Cu")
@@
 	)
 	(segment
-		(start 114.04746 127.173)
-		(end 105.84746 118.973)
+		(start 137.70486 120.713)
+		(end 135.09486 123.323)
 		(width 0.25)
 		(layer "B.Cu")
@@
 	)
 	(segment
-		(start 105.84746 45.373)
-		(end 114.49746 36.723)
+		(start 107.69746 113.223)
+		(end 105.84746 111.373)
+		(width 0.25)
+		(layer "B.Cu")
+		(net 44)
+	)
+	(segment
+		(start 179.04746 38.623)
+		(end 179.04746 40.473)
+		(width 0.25)
+		(layer "B.Cu")
+		(net 44)
+	)
+	(segment
+		(start 131.84746 123.323)
+		(end 130.22246 121.698)
+		(width 0.25)
+		(layer "B.Cu")
+		(net 44)
+	)
+	(segment
+		(start 135.09486 123.323)
+		(end 131.84746 123.323)
+		(width 0.25)
+		(layer "B.Cu")
+		(net 44)
+	)
+	(segment
+		(start 130.22246 114.848)
+		(end 128.59746 113.223)
 		(width 0.25)
 		(layer "B.Cu")
@@
 	)
 	(segment
-		(start 123.47246 107.873)
-		(end 123.49746 107.898)
-		(width 0.25)
-		(layer "B.Cu")
-		(net 227)
-	)
-	(segment
 		(start 203.67246 142.648)
 		(end 203.69746 142.623)
@@
 	)
 	(segment
-		(start 109.39746 89.223)
-		(end 113.99746 84.623)
+		(start 115.87246 106.998)
+		(end 114.29746 105.423)
 		(width 0.25)
 		(layer "B.Cu")
@@
 	)
 	(segment
-		(start 115.59746 107.873)
-		(end 113.99746 107.873)
+		(start 204.99746 142.655)
+		(end 204.96646 142.686)
 		(width 0.25)
 		(layer "B.Cu")
@@
 	)
 	(segment
-		(start 123.66246 107.733)
-		(end 123.49746 107.898)
+		(start 203.67246 142.773)
+		(end 203.67246 142.648)
 		(width 0.25)
 		(layer "B.Cu")
@@
 	)
 	(segment
-		(start 204.99746 142.655)
-		(end 204.96646 142.686)
+		(start 206.07746 135.793)
+		(end 204.99746 136.873)
 		(width 0.25)
 		(layer "B.Cu")
@@
 	)
 	(segment
-		(start 203.67246 142.773)
-		(end 203.67246 142.648)
+		(start 114.14746 84.473)
+		(end 113.99746 84.623)
 		(width 0.25)
 		(layer "B.Cu")
@@
 	)
 	(segment
-		(start 206.07746 135.793)
-		(end 204.99746 136.873)
+		(start 130.49746 107.733)
+		(end 123.98246 107.733)
 		(width 0.25)
 		(layer "B.Cu")
@@
 	)
 	(segment
-		(start 114.14746 84.473)
+		(start 109.39746 89.223)
 		(end 113.99746 84.623)
 		(width 0.25)
@@
 	)
 	(segment
-		(start 115.59746 107.873)
-		(end 123.47246 107.873)
+		(start 111.19746 105.423)
+		(end 109.39746 103.623)
 		(width 0.25)
 		(layer "B.Cu")
@@
 	)
 	(segment
-		(start 130.49746 107.733)
-		(end 123.66246 107.733)
+		(start 109.39746 103.623)
+		(end 109.39746 89.223)
 		(width 0.25)
 		(layer "B.Cu")
@@
 	)
 	(segment
-		(start 113.99746 107.873)
-		(end 109.39746 103.273)
+		(start 123.24746 106.998)
+		(end 115.87246 106.998)
+		(width 0.25)
+		(layer "B.Cu")
+		(net 227)
+	)
+	(segment
+		(start 114.29746 105.423)
+		(end 111.19746 105.423)
 		(width 0.25)
 		(layer "B.Cu")
@@
 	)
 	(segment
+		(start 123.98246 107.733)
+		(end 123.24746 106.998)
+		(width 0.25)
+		(layer "B.Cu")
+		(net 227)
+	)
+	(segment
 		(start 145.09746 84.473)
 		(end 114.14746 84.473)
@@
 	)
 	(segment
-		(start 109.39746 103.273)
-		(end 109.39746 89.223)
-		(width 0.25)
-		(layer "B.Cu")
-		(net 227)
-	)
-	(segment
 		(start 219.99746 99.573)
 		(end 208.24746 87.823)
@@
 		(name "$teardrop_padvia$")
 		(hatch full 0.1)
-		(priority 30002)
+		(priority 30000)
 		(attr
 			(teardrop
@@
 		(polygon
 			(pts
-				(xy 135.63037 83.293) (xy 135.63037 83.543) (xy 136.266357 83.842552) (xy 136.42043 83.473) (xy 136.266357 83.103448)
+				(xy 136.41943 84.248136) (xy 136.66943 84.248136) (xy 136.81943 83.473) (xy 136.41943 83.472) (xy 136.049878 83.626073)
 			)
 		)
@@
 		(name "$teardrop_padvia$")
 		(hatch full 0.1)
-		(priority 30001)
+		(priority 30002)
 		(attr
 			(teardrop
@@
 		(polygon
 			(pts
-				(xy 136.473504 96.795703) (xy 136.296727 96.618926) (xy 135.666357 96.903448) (xy 135.818723 97.273707)
-				(xy 136.188982 97.426073)
+				(xy 135.63037 83.293) (xy 135.63037 83.543) (xy 136.266357 83.842552) (xy 136.42043 83.473) (xy 136.266357 83.103448)
 			)
 		)
@@
 		(name "$teardrop_padvia$")
 		(hatch full 0.1)
-		(priority 30000)
+		(priority 30001)
 		(attr
 			(teardrop
@@
 		(polygon
 			(pts
-				(xy 136.41943 84.248136) (xy 136.66943 84.248136) (xy 136.81943 83.473) (xy 136.41943 83.472) (xy 136.049878 83.626073)
+				(xy 136.473504 96.795703) (xy 136.296727 96.618926) (xy 135.666357 96.903448) (xy 135.818723 97.273707)
+				(xy 136.188982 97.426073)
 			)
 		)
