File: rck.kicad_pcb (KiCad board)
At the start: 2 copper layers, 150 x 285 mm, 78 parts, among them J1 Conn_02x22_Row_Letter_Last, J2 Conn_02x22_Row_Letter_Last, J3 Conn_02x22_Row_Letter_Last, J4 Conn_02x22_Row_Letter_Last, J5 Conn_02x22_Row_Letter_Last, J6 Conn_02x22_Row_Letter_Last, J7 Conn_01x06_Pin

Commit message: 10F
Parts:
- moved C4 50.1 mm to (40.0, 36.6)
- moved C3 48.0 mm to (46.9, 41.3)
- moved C1 35.4 mm to (41.7, 49.6), turned to -90 degrees
- moved VR1 32.0 mm to (61.6, 45.0)
- moved C2 24.7 mm to (49.6, 48.9), turned to 90 degrees
- moved C8 9.57 mm to (128.3, 82.3)
- moved R11 9.37 mm to (78.5, 22.9)
- moved R14 9.37 mm to (91.3, 22.9)
- moved R17 9.37 mm to (104.1, 22.9)
- moved R2 9.37 mm to (40.0, 22.9)
- moved R23 9.37 mm to (129.8, 22.9)
- moved R26 9.37 mm to (142.6, 22.9)
- moved R5 9.37 mm to (52.8, 22.9)
- moved rD11 9.37 mm to (84.9, 22.9)
- moved rD14 9.37 mm to (97.7, 22.9)
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Connections:
- J1 pad 1a: VCC -> +5V
Routing:
- net VCC: track 152.9 -> 555.2 mm, vias 0 -> 2
- net /F9-01: track 0.05 -> 401.9 mm, vias 0 -> 1
- net /F9-02: track 0.00 -> 385.8 mm, vias 0 -> 1
- net /F10-01: track 0.00 -> 370.6 mm, vias 0 -> 1
- net /F9-03: track 0.00 -> 354.8 mm, vias 0 -> 1
- net /F10-02: track 0.00 -> 347.5 mm, vias 0 -> 1
- net /F10-03: track 0.00 -> 325.1 mm, vias 0 -> 1
- net /F7-01: track 0.00 -> 312.4 mm, vias 0 -> 5
- net /F7-03: track 0.00 -> 302.4 mm, vias 0 -> 1
- net /F7-02: track 0.00 -> 295.4 mm, vias 0 -> 5
- net /F8-01: track 0.00 -> 293.2 mm, vias 0 -> 1
- net /F8-02: track 0.00 -> 268.7 mm, vias 0 -> 1
- net /F8-03: track 0.00 -> 251.6 mm, vias 0 -> 1
- net +12V: track 18.5 -> 259.7 mm
- net /F5-01: track 0.00 -> 194.1 mm, vias 0 -> 4
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- added copper zone on B.Cu, net GND
- added copper zone on F.Cu, net GND
Other:
- board size 150 x 285 mm -> 150 x 295 mm

Commit message: change page size
Parts:
- moved C2 95.5 mm to (123.5, 109.4)
- moved C6 95.5 mm to (211.8, 137.3)
- moved J2 95.5 mm to (217.0, 155.6)
- moved R11 95.5 mm to (152.4, 83.4)
- moved R17 95.5 mm to (178.0, 83.4)
- moved R2 95.5 mm to (113.9, 83.4)
- moved R20 95.5 mm to (190.9, 83.4)
- moved R26 95.5 mm to (216.5, 83.4)
- moved R29 95.5 mm to (229.4, 83.4)
- moved R5 95.5 mm to (126.7, 83.4)
- moved rD11 95.5 mm to (158.8, 83.4)
- moved rD17 95.5 mm to (184.4, 83.4)
- moved rD2 95.5 mm to (120.3, 83.4)
- moved rD20 95.5 mm to (197.3, 83.4)
- moved rD26 95.5 mm to (222.9, 83.4)
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
Commit message: F10 Compleate
Parts:
- added Brd1: SSD1306, SSD1306:128x64OLED, F.Cu at (175.0, 51.1)
- added F1: SMD0805-020-16V - 2.8A, Fuse:Fuse_0805_2012Metric, B.Cu at (119.2, 58.4)
- added F2: SMD0805-020-16V - 500mA, Fuse:Fuse_0805_2012Metric, B.Cu at (114.0, 96.1)
- added F3: SMD0603-050 - 1A, Fuse:Fuse_0603_1608Metric, B.Cu at (202.2, 132.8)
- J7: value Conn_01x06_Pin -> Conn_01x02_Pin; footprint Connector_PinSocket_2.54mm:PinSocket_1x06_P2.54mm_Vertical -> Connector_PinSocket_2.54mm:PinSocket_1x02_P2.54mm_Vertical
- moved J7 17.6 mm to (119.2, 41.3)
- moved C6 8.28 mm to (203.5, 136.9)
- moved C7 7.61 mm to (193.9, 134.8)
- moved C5 7.52 mm to (202.8, 142.7)
- moved C8 7.52 mm to (194.7, 142.2)
- moved REF** 5.00 mm to (216.4, 147.2)
- moved VR2 5.00 mm to (212.4, 135.8)
- moved C4 3.37 mm to (113.5, 100.4), turned to 0 degrees
Connections:
- C1 pad 1: +12V -> Net-(VR1-Vin)
- C2 pad 2: +12V -> Net-(VR1-Vin)
- C3 pad 1: VCC -> Net-(VR1-Vout)
- C4 pad 2: VCC -> Net-(VR1-Vout)
- C5 pad 1: +12V -> Net-(VR1-Vin)
- C6 pad 2: +12V -> Net-(VR1-Vin)
- C7 pad 1: +5V -> Net-(VR2-Vout)
- C8 pad 2: +5V -> Net-(VR2-Vout)
- J1 pad 20b: unconnected-(J1-Pin_20b-Pad20b) -> /3V
- J1 pad 21b: unconnected-(J1-Pin_21b-Pad21b) -> /SDA
- J1 pad 22b: unconnected-(J1-Pin_22b-Pad22b) -> /SCL
- VR1 pad 1: +12V -> Net-(VR1-Vin)
- VR1 pad 3: VCC -> Net-(VR1-Vout)
- VR2 pad 1: +12V -> Net-(VR1-Vin)
- VR2 pad 3: +5V -> Net-(VR2-Vout)
Routing:
- net +12V: track 259.7 -> 16.2 mm
- net Net-(VR1-Vin): track 0.00 -> 238.5 mm
- net /3V: track 0.00 -> 191.8 mm, vias 0 -> 1
- net /SDA: track 0.00 -> 190.9 mm
- net /SCL: track 0.00 -> 176.4 mm
- net Net-(VR2-Vout): track 0.00 -> 35.4 mm
- net +5V: track 61.6 -> 28.0 mm
- net VCC: track 555.2 -> 527.2 mm
- net Net-(VR1-Vout): track 0.00 -> 22.8 mm
- net /F1-01: track 170.3 -> 176.5 mm
- net /F6-01: track 192.5 -> 194.5 mm
- net /F4-02: track 145.0 -> 143.3 mm
- net /F3-01: track 172.4 -> 173.7 mm
- net /F10-02: track 347.5 -> 348.6 mm
- net /F8-02: track 268.7 -> 267.6 mm
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Other:
- board size 150 x 295 mm -> 150 x 310.5 mm

Commit message: fix routes
Parts:
- moved C1 2.80 mm to (115.4, 107.3)
- moved C2 1.82 mm to (123.2, 107.6)
Routing:
- net /3V: track 191.8 -> 185.3 mm
- net /SCL: track 176.4 -> 170.3 mm
- net /SDA: track 190.9 -> 185.3 mm
- net /F6-01: track 194.5 -> 193.8 mm

Commit message: Delete vias
Routing:
- net /F4-03: track 137.8 -> 135.5 mm, vias 3 -> 2
- net /F6-03: track 183.7 -> 181.5 mm, vias 4 -> 3
- net /F2-03: track 179.8 -> 177.8 mm, vias 2 -> 1
- net /F6-01: track 193.8 -> 192.0 mm, vias 4 -> 3
- net /F6-02: track 186.2 -> 184.7 mm, vias 4 -> 3
- net /F7-01: track 312.3 -> 310.8 mm, vias 5 -> 4
- net /F4-01: track 147.3 -> 145.8 mm, vias 3 -> 2
- net /F5-01: track 194.1 -> 192.6 mm, vias 4 -> 3
- net /F4-02: track 143.3 -> 141.8 mm, vias 3 -> 2
- net /F3-01: track 173.7 -> 172.3 mm, vias 3 -> 2
- net /F3-03: track 139.6 -> 138.2 mm, vias 3 -> 2
- net /F3-02: track 153.9 -> 152.6 mm, vias 3 -> 2
- net /F5-02: track 174.8 -> 173.5 mm, vias 4 -> 3
- net /F7-02: track 295.4 -> 294.2 mm, vias 5 -> 4
- net /F5-03: track 163.4 -> 162.2 mm, vias 4 -> 3
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Other:
- board size 150 x 310.5 mm -> 150 x 325.6 mm
